File: PCB/LRA/LRAdriver/LRAdriver.kicad_sch (KiCad schematic)
At the start: 6 parts, among them J1 Conn_01x02_Pin, U1 DRV2605LTDGSRQ1

Commit message: ESP32 S2 schematic done.
Parts:
- R1, R2: value R_Small -> 2.2k
Changed lines of the file:
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@@
 			)
 		)
-		(property "Value" "R_Small"
+		(property "Value" "2.2k"
 			(at 115.57 95.25 90)
 			(effects
@@
 			)
 		)
-		(property "Value" "R_Small"
+		(property "Value" "2.2k"
 			(at 109.22 91.44 90)
 			(effects
