File: PCB/ESP32/ESP32/ESP32.kicad_sch (KiCad schematic)
At the start: 29 parts, among them J1 Conn_01x02_Pin, J1 USB_B_Micro, J2 Conn_01x02_Socket, SW1 RESET, SW2 BOOT, SW3 LRA Switch, U1 DRV2605LTDGSRQ1, U1 ESP32-S2-SOLO-U-N4, U1 MCP73832T-2ACI/OT

Commit message: done.
Parts:
- added D1: D_Schottky, symbol Device:D_Schottky
- added J1: Camera_Receptacle_THT, symbol Connector:DA15_Receptacle_MountingHoles
- renumbered C1 to C5, C4 to C6, C2 to C7, C3 to C8, C5 to C9, R1 to R7
Connections:
- net +3V3: now also J1.1 (3V3); no longer C2.1, J2.1 (Pin_1), U1.3
- net GND: now also J1.10 (GND)
- net SCL: now also J1.2 (SCL)
- net SDA: now also J1.11 (SDA)
- net D7: now reaches U1.12 (IO8)
- net D7: now also J1.5 (D7)
- net D2: now reaches U1.15 (IO3)
- net D2: now also J1.16 (D2)
- net PWNN: now reaches U1.20 (IO12)
- net PWNN: now also J1.18 (PWNN)
- net PCLK: now reaches U1.21 (IO13)
- net PCLK: now also J1.4 (PCLK)
- net MCLK: now reaches U1.22 (IO14)
- net MCLK: now also J1.13 (MCLK)
- net Reset: now reaches C5.2, R7.2, SW1.2 (B), U1.3 (EN)
- net Reset: now also J1.9 (RST)
- net D1: now reaches U1.38 (IO2)
- net D1: now also J1.8 (D1)
- net D0: now reaches U1.39 (IO1)
- net D0: now also J1.17 (D0)
- net D3: now reaches U1.4 (IO4)
- net D3: now also J1.7 (D3)
- net D4: now reaches U1.5 (IO5)
- net D4: now also J1.15 (D4)
- net D5: now reaches U1.6 (IO6)
- net D5: now also J1.6 (D5)
- net D6: now reaches U1.7 (IO7)
- net D6: now also J1.14 (D6)
- net VS: now reaches U1.8 (IO15)
- net VS: now also J1.3 (VS)
- net HS: now reaches U1.9 (IO16)
- net HS: now also J1.12 (HS)
- new net: D1.1 (K), J2.1 (Pin_1)
- new net: C2.1, D1.2 (A), U1.3
Other:
- note added: "Drop Voltage vy about .5V"
- moved on the sheet: C1, C2, D1, D2, J1, J2, JP1, JP2, R1, R2, R3, R4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

Commit message: Coworking test
Parts:
- added R8: R, symbol Device:R
Connections:
- net GND: now also R8.1
- net SCL: now also R8.2
Changed lines of the file:
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@@
 	(wire
 		(pts
-			(xy 309.88 110.49) (xy 311.15 110.49)
+			(xy 313.69 53.34) (xy 322.58 53.34)
 		)
 		(stroke
@@
 	(wire
 		(pts
-			(xy 313.69 53.34) (xy 322.58 53.34)
+			(xy 267.97 38.1) (xy 265.43 38.1)
 		)
 		(stroke
@@
 	(wire
 		(pts
-			(xy 267.97 38.1) (xy 265.43 38.1)
+			(xy 256.54 52.07) (xy 254 52.07)
 		)
 		(stroke
@@
 	(wire
 		(pts
-			(xy 256.54 52.07) (xy 254 52.07)
+			(xy 152.4 195.58) (xy 161.29 195.58)
 		)
 		(stroke
@@
 	(wire
 		(pts
-			(xy 152.4 195.58) (xy 161.29 195.58)
+			(xy 102.87 78.74) (xy 109.22 78.74)
 		)
 		(stroke
@@
 	(wire
 		(pts
-			(xy 102.87 78.74) (xy 109.22 78.74)
+			(xy 144.78 60.96) (xy 161.29 60.96)
 		)
 		(stroke
@@
 	(wire
 		(pts
-			(xy 144.78 60.96) (xy 161.29 60.96)
+			(xy 306.07 110.49) (xy 311.15 110.49)
 		)
 		(stroke
@@
 	(wire
 		(pts
+			(xy 298.45 110.49) (xy 292.1 110.49)
+		)
+		(stroke
+			(width 0)
+			(type default)
+		)
+	)
+	(wire
+		(pts
 			(xy 306.07 125.73) (xy 311.15 125.73)
 		)
@@
 	(wire
 		(pts
+			(xy 292.1 110.49) (xy 292.1 114.3)
+		)
+		(stroke
+			(width 0)
+			(type default)
+		)
+	)
+	(wire
+		(pts
 			(xy 309.88 113.03) (xy 311.15 113.03)
 		)
@@
 	(label "SDA"
 		(at 309.88 113.03 180)
+		(fields_autoplaced yes)
 		(effects
 			(font
@@
 	(label "D7"
 		(at 102.87 78.74 180)
+		(fields_autoplaced yes)
 		(effects
 			(font
@@
 	(label "SDA"
 		(at 273.05 53.34 270)
+		(fields_autoplaced yes)
 		(effects
 			(font
@@
 	(label "MCLK"
 		(at 306.07 123.19 180)
+		(fields_autoplaced yes)
 		(effects
 			(font
@@
 	(label "D1"
 		(at 306.07 140.97 180)
+		(fields_autoplaced yes)
 		(effects
 			(font
@@
 	(label "D3"
 		(at 105.41 69.85 180)
+		(fields_autoplaced yes)
 		(effects
 			(font
@@
 	(label "Reset"
 		(at 306.07 146.05 180)
+		(fields_autoplaced yes)
 		(effects
 			(font
@@
 	(label "SCL"
 		(at 309.88 110.49 180)
+		(fields_autoplaced yes)
 		(effects
 			(font
@@
 	(label "D5"
 		(at 306.07 130.81 180)
+		(fields_autoplaced yes)
 		(effects
 			(font
@@
 	(label "Reset"
 		(at 99.06 41.91 180)
+		(fields_autoplaced yes)
 		(effects
 			(font
@@
 	(label "D7"
 		(at 306.07 125.73 180)
+		(fields_autoplaced yes)
 		(effects
 			(font
@@
 	(label "D4"
 		(at 306.07 133.35 180)
+		(fields_autoplaced yes)
 		(effects
 			(font
@@
 	(label "PWNN"
 		(at 307.34 148.59 180)
+		(fields_autoplaced yes)
 		(effects
 			(font
@@
 	(label "VS"
 		(at 105.41 96.52 180)
+		(fields_autoplaced yes)
 		(effects
 			(font
@@
 	(label "D6"
 		(at 105.41 77.47 180)
+		(fields_autoplaced yes)
 		(effects
 			(font
@@
 	(label "USB_D+"
 		(at 45.72 198.12 0)
+		(fields_autoplaced yes)
 		(effects
 			(font
@@
 	(label "D6"
 		(at 306.07 128.27 180)
+		(fields_autoplaced yes)
 		(effects
 			(font
@@
 	(label "SCL"
 		(at 107.95 81.28 180)
+		(fields_autoplaced yes)
 		(effects
 			(font
@@
 	(label "D4"
 		(at 105.41 72.39 180)
+		(fields_autoplaced yes)
 		(effects
 			(font
@@
 	(label "MCLK"
 		(at 105.41 93.98 180)
+		(fields_autoplaced yes)
 		(effects
 			(font
@@
 	(label "D0"
 		(at 105.41 62.23 180)
+		(fields_autoplaced yes)
 		(effects
 			(font
@@
 	(label "D3"
 		(at 306.07 135.89 180)
+		(fields_autoplaced yes)
 		(effects
 			(font
@@
 	(label "USB_D-"
 		(at 148.59 63.5 0)
+		(fields_autoplaced yes)
 		(effects
 			(font
@@
 	(label "PWNN"
 		(at 102.87 88.9 180)
+		(fields_autoplaced yes)
 		(effects
 			(font
@@
 	(label "D0"
 		(at 306.07 143.51 180)
+		(fields_autoplaced yes)
 		(effects
 			(font
@@
 	(label "D2"
 		(at 306.07 138.43 180)
+		(fields_autoplaced yes)
 		(effects
 			(font
@@
 	(label "USB_D+"
 		(at 148.59 66.04 0)
+		(fields_autoplaced yes)
 		(effects
 			(font
@@
 	(label "SDA"
 		(at 107.95 83.82 180)
+		(fields_autoplaced yes)
 		(effects
 			(font
@@
 	(label "VS"
 		(at 309.88 115.57 180)
+		(fields_autoplaced yes)
 		(effects
 			(font
@@
 	(label "PCLK"
 		(at 104.14 91.44 180)
+		(fields_autoplaced yes)
 		(effects
 			(font
@@
 	(label "USB_D-"
 		(at 45.72 200.66 0)
+		(fields_autoplaced yes)
 		(effects
 			(font
@@
 	(label "D1"
 		(at 105.41 64.77 180)
+		(fields_autoplaced yes)
 		(effects
 			(font
@@
 	(label "HS"
 		(at 308.61 118.11 180)
+		(fields_autoplaced yes)
 		(effects
 			(font
@@
 	(label "PCLK"
 		(at 307.34 120.65 180)
+		(fields_autoplaced yes)
 		(effects
 			(font
@@
 	(label "D2"
 		(at 105.41 67.31 180)
+		(fields_autoplaced yes)
 		(effects
 			(font
@@
 	(label "D5"
 		(at 105.41 74.93 180)
+		(fields_autoplaced yes)
 		(effects
 			(font
@@
 	(label "HS"
 		(at 148.59 55.88 0)
+		(fields_autoplaced yes)
 		(effects
 			(font
@@
 	(label "SCL"
 		(at 271.78 46.99 270)
+		(fields_autoplaced yes)
 		(effects
 			(font
@@
 	)
 	(symbol
+		(lib_id "Device:R")
+		(at 302.26 110.49 90)
+		(unit 1)
+		(exclude_from_sim no)
+		(in_bom yes)
+		(on_board yes)
+		(dnp no)
+		(fields_autoplaced yes)
+		(property "Reference" "R8"
+			(at 302.26 104.14 90)
+			(effects
+				(font
+					(size 1.27 1.27)
+				)
+			)
+		)
+		(property "Value" "R"
+			(at 302.26 106.68 90)
+			(effects
+				(font
+					(size 1.27 1.27)
+				)
+			)
+		)
+		(property "Footprint" ""
+			(at 302.26 112.268 90)
+			(effects
+				(font
+					(size 1.27 1.27)
+				)
+				(hide yes)
+			)
+		)
+		(property "Datasheet" "~"
+			(at 302.26 110.49 0)
+			(effects
+				(font
+					(size 1.27 1.27)
+				)
+				(hide yes)
+			)
+		)
+		(property "Description" "Resistor"
+			(at 302.26 110.49 0)
+			(effects
+				(font
+					(size 1.27 1.27)
+				)
+				(hide yes)
+			)
+		)
+		(pin "2"
+		)
+		(pin "1"
+		)
+		(instances
+			(project ""
+				(path "/f9099a9a-ca12-4d9e-a4e7-b3f085e605c9"
+					(reference "R8")
+					(unit 1)
+				)
+			)
+		)
+	)
+	(symbol
 		(lib_id "power:GND")
 		(at 173.99 35.56 0)
@@
 					(unit 1)
 				)
+			)
+		)
+	)
+	(symbol
+		(lib_id "power:GND")
+		(at 292.1 114.3 0)
+		(unit 1)
+		(exclude_from_sim no)
+		(in_bom yes)
+		(on_board yes)
+		(dnp no)
+		(fields_autoplaced yes)
+		(property "Reference" "#PWR010"
+			(at 292.1 120.65 0)
+			(effects
+				(font
+					(size 1.27 1.27)
+				)
+				(hide yes)
+			)
+		)
+		(property "Value" "GND"
+			(at 292.1 119.38 0)
+			(effects
+				(font
+					(size 1.27 1.27)
+				)
+			)
+		)
+		(property "Footprint" ""
+			(at 292.1 114.3 0)
+			(effects
+				(font
+					(size 1.27 1.27)
+				)
+				(hide yes)
+			)
+		)
+		(property "Datasheet" ""
+			(at 292.1 114.3 0)
+			(effects
+				(font
+					(size 1.27 1.27)
+				)
+				(hide yes)
+			)
+		)
+		(property "Description" "Power symbol creates a global label with name \"GND\" , ground"
+			(at 292.1 114.3 0)
+			(effects
+				(font
+					(size 1.27 1.27)
+				)
+				(hide yes)
+			)
+		)
+		(pin "1"
+		)
+		(instances
+			(project ""
+				(path "/f9099a9a-ca12-4d9e-a4e7-b3f085e605c9"
+					(reference "#PWR010")
+					(unit 1)
+				)

Commit message: test
Parts:
- removed R8: R, symbol Device:R
Connections:
- net SCL: no longer J1.2 (SCL)
- net SDA: no longer J1.11 (SDA)

Commit message: test
Parts:
- added R8: R, symbol Device:R
Connections:
- net GND: now also R8.2
- net at J1.2 (SCL): now also R8.1
Changed lines of the file:
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@@
 	(wire
 		(pts
+			(xy 287.02 110.49) (xy 287.02 114.3)
+		)
+		(stroke
+			(width 0)
+			(type default)
+		)
+	)
+	(wire
+		(pts
 			(xy 313.69 35.56) (xy 313.69 33.02)
 		)
@@
 	(label "D7"
 		(at 102.87 78.74 180)
+		(fields_autoplaced yes)
 		(effects
 			(font
@@
 	(label "SDA"
 		(at 273.05 53.34 270)
+		(fields_autoplaced yes)
 		(effects
 			(font
@@
 	(label "MCLK"
 		(at 306.07 123.19 180)
+		(fields_autoplaced yes)
 		(effects
 			(font
@@
 	(label "D1"
 		(at 306.07 140.97 180)
+		(fields_autoplaced yes)
 		(effects
 			(font
@@
 	(label "D3"
 		(at 105.41 69.85 180)
+		(fields_autoplaced yes)
 		(effects
 			(font
@@
 	(label "Reset"
 		(at 306.07 146.05 180)
+		(fields_autoplaced yes)
 		(effects
 			(font
@@
 	(label "D5"
 		(at 306.07 130.81 180)
+		(fields_autoplaced yes)
 		(effects
 			(font
@@
 	(label "Reset"
 		(at 99.06 41.91 180)
+		(fields_autoplaced yes)
 		(effects
 			(font
@@
 	(label "D7"
 		(at 306.07 125.73 180)
+		(fields_autoplaced yes)
 		(effects
 			(font
@@
 	(label "D4"
 		(at 306.07 133.35 180)
+		(fields_autoplaced yes)
 		(effects
 			(font
@@
 	(label "PWNN"
 		(at 307.34 148.59 180)
+		(fields_autoplaced yes)
 		(effects
 			(font
@@
 	(label "VS"
 		(at 105.41 96.52 180)
+		(fields_autoplaced yes)
 		(effects
 			(font
@@
 	(label "D6"
 		(at 105.41 77.47 180)
+		(fields_autoplaced yes)
 		(effects
 			(font
@@
 	(label "USB_D+"
 		(at 45.72 198.12 0)
+		(fields_autoplaced yes)
 		(effects
 			(font
@@
 	(label "D6"
 		(at 306.07 128.27 180)
+		(fields_autoplaced yes)
 		(effects
 			(font
@@
 	(label "SCL"
 		(at 107.95 81.28 180)
+		(fields_autoplaced yes)
 		(effects
 			(font
@@
 	(label "D4"
 		(at 105.41 72.39 180)
+		(fields_autoplaced yes)
 		(effects
 			(font
@@
 	(label "MCLK"
 		(at 105.41 93.98 180)
+		(fields_autoplaced yes)
 		(effects
 			(font
@@
 	(label "D0"
 		(at 105.41 62.23 180)
+		(fields_autoplaced yes)
 		(effects
 			(font
@@
 	(label "D3"
 		(at 306.07 135.89 180)
+		(fields_autoplaced yes)
 		(effects
 			(font
@@
 	(label "USB_D-"
 		(at 148.59 63.5 0)
+		(fields_autoplaced yes)
 		(effects
 			(font
@@
 	(label "PWNN"
 		(at 102.87 88.9 180)
+		(fields_autoplaced yes)
 		(effects
 			(font
@@
 	(label "D0"
 		(at 306.07 143.51 180)
+		(fields_autoplaced yes)
 		(effects
 			(font
@@
 	(label "D2"
 		(at 306.07 138.43 180)
+		(fields_autoplaced yes)
 		(effects
 			(font
@@
 	(label "USB_D+"
 		(at 148.59 66.04 0)
+		(fields_autoplaced yes)
 		(effects
 			(font
@@
 	(label "SDA"
 		(at 107.95 83.82 180)
+		(fields_autoplaced yes)
 		(effects
 			(font
@@
 	(label "VS"
 		(at 309.88 115.57 180)
+		(fields_autoplaced yes)
 		(effects
 			(font
@@
 	(label "PCLK"
 		(at 104.14 91.44 180)
+		(fields_autoplaced yes)
 		(effects
 			(font
@@
 	(label "USB_D-"
 		(at 45.72 200.66 0)
+		(fields_autoplaced yes)
 		(effects
 			(font
@@
 	(label "D1"
 		(at 105.41 64.77 180)
+		(fields_autoplaced yes)
 		(effects
 			(font
@@
 	(label "HS"
 		(at 308.61 118.11 180)
+		(fields_autoplaced yes)
 		(effects
 			(font
@@
 	(label "PCLK"
 		(at 307.34 120.65 180)
+		(fields_autoplaced yes)
 		(effects
 			(font
@@
 	(label "D2"
 		(at 105.41 67.31 180)
+		(fields_autoplaced yes)
+		(effects
+			(font
+				(size 1.27 1.27)
+			)
+			(justify right bottom)
+		)
+	)
+	(label "SCLK"
+		(at 287.02 114.3 180)
+		(fields_autoplaced yes)
 		(effects
 			(font
@@
 	(label "D5"
 		(at 105.41 74.93 180)
+		(fields_autoplaced yes)
 		(effects
 			(font
@@
 	(label "HS"
 		(at 148.59 55.88 0)
+		(fields_autoplaced yes)
 		(effects
 			(font
@@
 	(label "SCL"
 		(at 271.78 46.99 270)
+		(fields_autoplaced yes)
 		(effects
 			(font
@@
 	)
 	(symbol
+		(lib_id "Device:R")
+		(at 290.83 110.49 270)
+		(unit 1)
+		(exclude_from_sim no)
+		(in_bom yes)
+		(on_board yes)
+		(dnp no)
+		(fields_autoplaced yes)
+		(property "Reference" "R8"
+			(at 290.83 104.14 90)
+			(effects
+				(font
+					(size 1.27 1.27)
+				)
+			)
+		)
+		(property "Value" "R"
+			(at 290.83 106.68 90)
+			(effects
+				(font
+					(size 1.27 1.27)
+				)
+			)
+		)
+		(property "Footprint" ""
+			(at 290.83 108.712 90)
+			(effects
+				(font
+					(size 1.27 1.27)
+				)
+				(hide yes)
+			)
+		)
+		(property "Datasheet" "~"
+			(at 290.83 110.49 0)
+			(effects
+				(font
+					(size 1.27 1.27)
+				)
+				(hide yes)
+			)
+		)
+		(property "Description" "Resistor"
+			(at 290.83 110.49 0)
+			(effects
+				(font
+					(size 1.27 1.27)
+				)
+				(hide yes)
+			)
+		)
+		(pin "1"
+		)
+		(pin "2"
+		)
+		(instances
+			(project ""
+				(path "/f9099a9a-ca12-4d9e-a4e7-b3f085e605c9"
+					(reference "R8")
+					(unit 1)
+				)
+			)
+		)
+	)
+	(symbol
 		(lib_id "power:GND")
 		(at 175.26 212.09 0)
@@
 					(unit 1)
 				)
+			)
+		)
+	)
+	(symbol
+		(lib_id "power:GND")
+		(at 287.02 114.3 0)
+		(unit 1)
+		(exclude_from_sim no)
+		(in_bom yes)
+		(on_board yes)
+		(dnp no)
+		(fields_autoplaced yes)
+		(property "Reference" "#PWR010"
+			(at 287.02 120.65 0)
+			(effects
+				(font
+					(size 1.27 1.27)
+				)
+				(hide yes)
+			)
+		)
+		(property "Value" "GND"
+			(at 287.02 119.38 0)
+			(effects
+				(font
+					(size 1.27 1.27)
+				)
+			)
+		)
+		(property "Footprint" ""
+			(at 287.02 114.3 0)
+			(effects
+				(font
+					(size 1.27 1.27)
+				)
+				(hide yes)
+			)
+		)
+		(property "Datasheet" ""
+			(at 287.02 114.3 0)
+			(effects
+				(font
+					(size 1.27 1.27)
+				)
+				(hide yes)
+			)
+		)
+		(property "Description" "Power symbol creates a global label with name \"GND\" , ground"
+			(at 287.02 114.3 0)
+			(effects
+				(font
+					(size 1.27 1.27)
+				)
+				(hide yes)
+			)
+		)
+		(pin "1"
+		)
+		(instances
+			(project ""
+				(path "/f9099a9a-ca12-4d9e-a4e7-b3f085e605c9"
+					(reference "#PWR010")
+					(unit 1)
+				)

Commit message: Prelim footprints
Parts:
- J1: footprint (none) -> USB_Micro:CONN_10118193-0001LF_AMP
Changed lines of the file:
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@@
 			)
 		)
-		(property "Footprint" ""
+		(property "Footprint" "USB_Micro:CONN_10118193-0001LF_AMP"
 			(at 41.91 199.39 0)
 			(effects
