File: PCB/ESP32/ESP32/ESP32.kicad_sch (KiCad schematic)
At the start: 31 parts, among them J1 Camera_Receptacle_THT, J1 Conn_01x02_Pin, J1 USB_B_Micro, J2 Conn_01x02_Socket, SW1 RESET, SW2 BOOT, SW3 LRA Switch, U1 DRV2605LTDGSRQ1, U1 ESP32-S2-SOLO-U-N4, U1 MCP73832T-2ACI/OT

Commit message: Footprints finished
Finished JST, LRA footprint assignment
Parts:
- J1: footprint (none) -> ESP32_sym_footprint:CONN2_B2B-PH-K-S_JST
- J2: footprint Connector_JST:JST_GH_BM02B-GHS-TBT_1x02-1MP_P1.25mm_Vertical -> ESP32_sym_footprint:CONN2_B2B-PH-K-S_JST
- R7: footprint (none) -> Resistor_SMD:R_0805_2012Metric
- SW1, SW2, SW3: footprint (none) -> ESP32_sym_footprint:SW_TL59AF160Q_EWI
Changed lines of the file:
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@@
 	(label "D7"
 		(at 102.87 78.74 180)
-		(fields_autoplaced yes)
 		(effects
 			(font
@@
 	(label "SDA"
 		(at 273.05 53.34 270)
-		(fields_autoplaced yes)
 		(effects
 			(font
@@
 	(label "MCLK"
 		(at 306.07 123.19 180)
-		(fields_autoplaced yes)
 		(effects
 			(font
@@
 	(label "D1"
 		(at 306.07 140.97 180)
-		(fields_autoplaced yes)
 		(effects
 			(font
@@
 	(label "D3"
 		(at 105.41 69.85 180)
-		(fields_autoplaced yes)
 		(effects
 			(font
@@
 	(label "Reset"
 		(at 306.07 146.05 180)
-		(fields_autoplaced yes)
 		(effects
 			(font
@@
 	(label "D5"
 		(at 306.07 130.81 180)
-		(fields_autoplaced yes)
 		(effects
 			(font
@@
 	(label "Reset"
 		(at 99.06 41.91 180)
-		(fields_autoplaced yes)
 		(effects
 			(font
@@
 	(label "D7"
 		(at 306.07 125.73 180)
-		(fields_autoplaced yes)
 		(effects
 			(font
@@
 	(label "D4"
 		(at 306.07 133.35 180)
-		(fields_autoplaced yes)
 		(effects
 			(font
@@
 	(label "PWNN"
 		(at 307.34 148.59 180)
-		(fields_autoplaced yes)
 		(effects
 			(font
@@
 	(label "VS"
 		(at 105.41 96.52 180)
-		(fields_autoplaced yes)
 		(effects
 			(font
@@
 	(label "D6"
 		(at 105.41 77.47 180)
-		(fields_autoplaced yes)
 		(effects
 			(font
@@
 	(label "USB_D+"
 		(at 45.72 198.12 0)
-		(fields_autoplaced yes)
 		(effects
 			(font
@@
 	(label "D6"
 		(at 306.07 128.27 180)
-		(fields_autoplaced yes)
 		(effects
 			(font
@@
 	(label "SCL"
 		(at 107.95 81.28 180)
-		(fields_autoplaced yes)
 		(effects
 			(font
@@
 	(label "D4"
 		(at 105.41 72.39 180)
-		(fields_autoplaced yes)
 		(effects
 			(font
@@
 	(label "MCLK"
 		(at 105.41 93.98 180)
-		(fields_autoplaced yes)
 		(effects
 			(font
@@
 	(label "D0"
 		(at 105.41 62.23 180)
-		(fields_autoplaced yes)
 		(effects
 			(font
@@
 	(label "D3"
 		(at 306.07 135.89 180)
-		(fields_autoplaced yes)
 		(effects
 			(font
@@
 	(label "USB_D-"
 		(at 148.59 63.5 0)
-		(fields_autoplaced yes)
 		(effects
 			(font
@@
 	(label "PWNN"
 		(at 102.87 88.9 180)
-		(fields_autoplaced yes)
 		(effects
 			(font
@@
 	(label "D0"
 		(at 306.07 143.51 180)
-		(fields_autoplaced yes)
 		(effects
 			(font
@@
 	(label "D2"
 		(at 306.07 138.43 180)
-		(fields_autoplaced yes)
 		(effects
 			(font
@@
 	(label "USB_D+"
 		(at 148.59 66.04 0)
-		(fields_autoplaced yes)
 		(effects
 			(font
@@
 	(label "SDA"
 		(at 107.95 83.82 180)
-		(fields_autoplaced yes)
 		(effects
 			(font
@@
 	(label "VS"
 		(at 309.88 115.57 180)
-		(fields_autoplaced yes)
 		(effects
 			(font
@@
 	(label "PCLK"
 		(at 104.14 91.44 180)
-		(fields_autoplaced yes)
 		(effects
 			(font
@@
 	(label "USB_D-"
 		(at 45.72 200.66 0)
-		(fields_autoplaced yes)
 		(effects
 			(font
@@
 	(label "D1"
 		(at 105.41 64.77 180)
-		(fields_autoplaced yes)
 		(effects
 			(font
@@
 	(label "HS"
 		(at 308.61 118.11 180)
-		(fields_autoplaced yes)
 		(effects
 			(font
@@
 	(label "PCLK"
 		(at 307.34 120.65 180)
-		(fields_autoplaced yes)
 		(effects
 			(font
@@
 	(label "D2"
 		(at 105.41 67.31 180)
-		(fields_autoplaced yes)
 		(effects
 			(font
@@
 	(label "D5"
 		(at 105.41 74.93 180)
-		(fields_autoplaced yes)
 		(effects
 			(font
@@
 	(label "HS"
 		(at 148.59 55.88 0)
-		(fields_autoplaced yes)
 		(effects
 			(font
@@
 	(label "SCL"
 		(at 271.78 46.99 270)
-		(fields_autoplaced yes)
 		(effects
 			(font
@@
 			)
 		)
-		(property "Footprint" ""
+		(property "Footprint" "ESP32_sym_footprint:CONN2_B2B-PH-K-S_JST"
 			(at 328.93 30.48 0)
 			(effects
@@
 			)
 		)
-		(property "Footprint" ""
+		(property "Footprint" "ESP32_sym_footprint:SW_TL59AF160Q_EWI"
 			(at 166.37 60.96 0)
 			(effects
@@
 			)
 		)
-		(property "Footprint" ""
+		(property "Footprint" "ESP32_sym_footprint:SW_TL59AF160Q_EWI"
 			(at 90.17 45.72 0)
 			(effects
@@
 			)
 		)
-		(property "Footprint" ""
+		(property "Footprint" "Resistor_SMD:R_0805_2012Metric"
 			(at 104.14 43.18 0)
 			(effects
@@
 			)
 		)
-		(property "Footprint" ""
+		(property "Footprint" "ESP32_sym_footprint:SW_TL59AF160Q_EWI"
 			(at 93.98 59.69 0)
 			(effects
@@
 			)
 		)
-		(property "Footprint" "Connector_JST:JST_GH_BM02B-GHS-TBT_1x02-1MP_P1.25mm_Vertical"
+		(property "Footprint" "ESP32_sym_footprint:CONN2_B2B-PH-K-S_JST"
 			(at 208.28 186.69 0)
 			(effects

Commit message: Updated footprints for imported circuits
done
Parts:
- U1: footprint ESP32-S2-SOLO-U-N4:XCVR_ESP32-S2-SOLO-U-N4 -> ESP32_sym_footprint:XCVR_ESP32-S2-SOLO-U-N4
- U1: footprint SOT-23-5_MC_MCH -> ESP32_sym_footprint:SOT-23-5_MC_MCH
Changed lines of the file:
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@@
 			)
 		)
-		(property "Footprint" "ESP32-S2-SOLO-U-N4:XCVR_ESP32-S2-SOLO-U-N4"
+		(property "Footprint" "ESP32_sym_footprint:XCVR_ESP32-S2-SOLO-U-N4"
 			(at 127 71.12 0)
 			(effects
@@
 			)
 		)
-		(property "Footprint" "SOT-23-5_MC_MCH"
+		(property "Footprint" "ESP32_sym_footprint:SOT-23-5_MC_MCH"
 			(at 126.492 182.372 0)
 			(effects

Commit message: jhgj
Parts:
- D1: footprint Schottky_Diode_Battery:DO-41_STM -> ESP32_sym_footprint:DO-41_STM
- J1: footprint USB_Micro:CONN_10118193-0001LF_AMP -> ESP32_sym_footprint:CONN_10118193-0001LF_AMP
- U1: footprint DGS0010A_N -> ESP32_sym_footprint:DGS0010A_L
Changed lines of the file:
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@@
 			)
 		)
-		(property "Footprint" "USB_Micro:CONN_10118193-0001LF_AMP"
+		(property "Footprint" "ESP32_sym_footprint:CONN_10118193-0001LF_AMP"
 			(at 41.91 199.39 0)
 			(effects
@@
 			)
 		)
-		(property "Footprint" "Schottky_Diode_Battery:DO-41_STM"
+		(property "Footprint" "ESP32_sym_footprint:DO-41_STM"
 			(at 195.58 186.69 0)
 			(effects
@@
 			)
 		)
-		(property "Footprint" "DGS0010A_N"
+		(property "Footprint" "ESP32_sym_footprint:DGS0010A_L"
 			(at 293.37 40.64 0)
 			(effects
