File: PCB/ESP32/ESP32/_autosave-ESP32.kicad_sch (KiCad schematic)
At the start: 40 parts, among them J1 Conn_01x02_Pin, J1 PPTC091LFBN-RC, J2 PPTC091LFBN-RC, J4 Conn_01x02_Socket, J5 USB_B_Micro, Q1 PMOS, SW1 RESET, SW2 BOOT, SW3 LRA Switch, U1 DRV2605LTDGSRQ1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

Commit message: WIP of the new layout.
Parts:
- D1: footprint Footprint:DO-41_STM -> Schottky_Diode_Battery:CR_SMA_403AE_OSI-L
- U2: footprint Footprint:XCVR_ESP32-S2-SOLO-U-N4 -> ESP32_sym_footprint:XCVR_ESP32-S2-SOLO-N4
Changed lines of the file:
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@@
 	(label "D7"
 		(at 102.87 78.74 180)
+		(fields_autoplaced yes)
 		(effects
 			(font
@@
 	(label "USB_D+"
 		(at 81.28 212.09 0)
+		(fields_autoplaced yes)
 		(effects
 			(font
@@
 	(label "SDA"
 		(at 273.05 53.34 270)
+		(fields_autoplaced yes)
 		(effects
 			(font
@@
 	(label "SDA"
 		(at 316.23 119.38 0)
+		(fields_autoplaced yes)
 		(effects
 			(font
@@
 	(label "D6"
 		(at 298.45 127 0)
+		(fields_autoplaced yes)
 		(effects
 			(font
@@
 	(label "D3"
 		(at 105.41 69.85 180)
+		(fields_autoplaced yes)
 		(effects
 			(font
@@
 	(label "D0"
 		(at 298.45 134.62 0)
+		(fields_autoplaced yes)
 		(effects
 			(font
@@
 	(label "VS"
 		(at 105.41 96.52 180)
+		(fields_autoplaced yes)
 		(effects
 			(font
@@
 	(label "USB_D-"
 		(at 81.28 214.63 0)
+		(fields_autoplaced yes)
 		(effects
 			(font
@@
 	(label "D6"
 		(at 105.41 77.47 180)
+		(fields_autoplaced yes)
 		(effects
 			(font
@@
 	(label "D7"
 		(at 259.08 127 180)
+		(fields_autoplaced yes)
 		(effects
 			(font
@@
 	(label "D5"
 		(at 259.08 129.54 180)
+		(fields_autoplaced yes)
 		(effects
 			(font
@@
 	(label "VS"
 		(at 259.08 121.92 180)
+		(fields_autoplaced yes)
 		(effects
 			(font
@@
 	(label "MCLK"
 		(at 331.47 124.46 0)
+		(fields_autoplaced yes)
 		(effects
 			(font
@@
 	(label "SCL"
 		(at 107.95 81.28 180)
+		(fields_autoplaced yes)
 		(effects
 			(font
@@
 	(label "D4"
 		(at 105.41 72.39 180)
+		(fields_autoplaced yes)
 		(effects
 			(font
@@
 	(label "SCL"
 		(at 240.03 119.38 180)
+		(fields_autoplaced yes)
 		(effects
 			(font
@@
 	(label "MCLK"
 		(at 105.41 93.98 180)
+		(fields_autoplaced yes)
 		(effects
 			(font
@@
 	(label "D0"
 		(at 105.41 62.23 180)
+		(fields_autoplaced yes)
 		(effects
 			(font
@@
 	(label "D2"
 		(at 298.45 132.08 0)
+		(fields_autoplaced yes)
 		(effects
 			(font
@@
 	(label "USB_D-"
 		(at 148.59 63.5 0)
+		(fields_autoplaced yes)
 		(effects
 			(font
@@
 	(label "USB_D+"
 		(at 148.59 66.04 0)
+		(fields_autoplaced yes)
 		(effects
 			(font
@@
 	(label "PCLK"
 		(at 259.08 124.46 180)
+		(fields_autoplaced yes)
 		(effects
 			(font
@@
 	(label "SDA"
 		(at 107.95 83.82 180)
+		(fields_autoplaced yes)
 		(effects
 			(font
@@
 	(label "PCLK"
 		(at 104.14 91.44 180)
+		(fields_autoplaced yes)
 		(effects
 			(font
@@
 	(label "D4"
 		(at 298.45 129.54 0)
+		(fields_autoplaced yes)
 		(effects
 			(font
@@
 	(label "D1"
 		(at 105.41 64.77 180)
+		(fields_autoplaced yes)
 		(effects
 			(font
@@
 	(label "D1"
 		(at 259.08 134.62 180)
+		(fields_autoplaced yes)
 		(effects
 			(font
@@
 	(label "D2"
 		(at 105.41 67.31 180)
+		(fields_autoplaced yes)
 		(effects
 			(font
@@
 	(label "D3"
 		(at 259.08 132.08 180)
+		(fields_autoplaced yes)
 		(effects
 			(font
@@
 	(label "HS"
 		(at 298.45 121.92 0)
+		(fields_autoplaced yes)
 		(effects
 			(font
@@
 	(label "D5"
 		(at 105.41 74.93 180)
+		(fields_autoplaced yes)
 		(effects
 			(font
@@
 	(label "HS"
 		(at 148.59 55.88 0)
+		(fields_autoplaced yes)
 		(effects
 			(font
@@
 	(label "SCL"
 		(at 271.78 46.99 270)
+		(fields_autoplaced yes)
 		(effects
 			(font
@@
 			)
 		)
-		(property "Footprint" "Footprint:XCVR_ESP32-S2-SOLO-U-N4"
+		(property "Footprint" "ESP32_sym_footprint:XCVR_ESP32-S2-SOLO-N4"
 			(at 127 71.12 0)
 			(effects
@@
 			)
 		)
-		(property "Footprint" "Footprint:DO-41_STM"
+		(property "Footprint" "Schottky_Diode_Battery:CR_SMA_403AE_OSI-L"
 			(at 187.96 195.58 0)
 			(effects
@@
 			)
 		)
-		(property "Footprint" "Footprint:DO-41_STM"
+		(property "Footprint" "Schottky_Diode_Battery:CR_SMA_403AE_OSI-L"
 			(at 187.96 184.15 0)
 			(effects
