File: PCB/ESP32/ESP32/ESP32.kicad_pcb (KiCad board)
At the start: 2 copper layers, 51 x 51 mm, 40 parts, among them J1 PPTC091LFBN-RC, J2 PPTC091LFBN-RC, U2 ESP32-S2-SOLO-U-N4

Commit message: WIP of the new layout.
Parts:
- removed Charge IC: MCP73832T-2ACI/OT, Footprint:SOT-23-5_MC_MCH
- added REF**: MountingHole_3.2mm_M3, MountingHole:MountingHole_3.2mm_M3, F.Cu at (138.5, 147.7)
- added REF**: MountingHole_3.2mm_M3, MountingHole:MountingHole_3.2mm_M3, F.Cu at (115.2, 148.1)
- added REF**: MountingHole_3.2mm_M3, MountingHole:MountingHole_3.2mm_M3, F.Cu at (115.3, 113.0)
- added REF**: MountingHole_3.2mm_M3, MountingHole:MountingHole_3.2mm_M3, F.Cu at (138.7, 112.8)
- C10, C12, C13, C8, C9, D4, D5, JP2, R1, R10, R12, R13, R17, R18, R19, R2, R4, R5, R8: moved to B.Cu
- D1, D6: footprint Footprint:DO-41_STM -> Schottky_Diode_Battery:CR_SMA_403AE_OSI-L; moved to B.Cu
- J3: renamed from LRA pins; moved to B.Cu
- J4: renamed from Bat pins; moved to B.Cu
- J5: renamed from USB; moved to B.Cu
- Q1: renamed from PMOS; moved to B.Cu
- U2: footprint Footprint:XCVR_ESP32-S2-SOLO-U-N4 -> ESP32_sym_footprint:XCVR_ESP32-S2-SOLO-N4
- U5: renamed from LRA driver; moved to B.Cu
- U6: renamed from LDO; moved to B.Cu
- moved C2 80.1 mm to (133.5, 110.8), turned to 180 degrees
- moved SW1 79.7 mm to (132.8, 114.2)
- moved R3 79.2 mm to (133.5, 109.1), turned to 180 degrees
- moved U2 76.9 mm to (129.2, 126.7)
- moved C4 72.7 mm to (129.2, 154.4)
- moved C5 72.7 mm to (133.5, 154.5)
- moved C3 70.4 mm to (117.1, 140.6), turned to 0 degrees
- moved C6 68.9 mm to (128.7, 149.5), turned to 90 degrees
- moved R2 68.4 mm to (121.8, 111.5), turned to 90 degrees
- moved R4 68.4 mm to (121.8, 115.0)
- moved SW3 65.3 mm to (126.0, 146.5)
- moved J1 65.2 mm to (117.0, 104.1)
- moved J2 65.2 mm to (117.0, 106.6)
- moved R1 64.8 mm to (115.2, 133.3), turned to 180 degrees
- moved J3 64.3 mm to (113.8, 121.0), turned to -90 degrees
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- renumbered RES to SW1, BOOT to SW2, LRA_test to SW3
Connections:
- net 5V renamed Net-(D4-A)
- net Charge-line renamed Net-(J4-Pin_1)
Routing:
- net GND: track 137.4 -> 11.3 mm, vias 13 -> 0
- net /PCLK: track 68.9 -> 30.3 mm, vias 2 -> 1
- net /VS: track 42.3 -> 15.3 mm
- net /D1: track 54.3 -> 32.5 mm, vias 0 -> 1
- net +3V3: track 27.7 -> 6.19 mm, vias 13 -> 0
- net /SCL: track 59.7 -> 39.1 mm, vias 0 -> 1
- net /HS: track 32.6 -> 12.2 mm, vias 2 -> 0
- net /D5: track 33.5 -> 14.5 mm
- net /D0: track 47.8 -> 29.5 mm, vias 2 -> 1
- net /D6: track 29.7 -> 11.4 mm
- net /D4: track 29.7 -> 11.4 mm
- net /D3: track 32.4 -> 14.5 mm
- net /USB_D+: track 42.9 -> 26.7 mm, vias 2 -> 1
- net /D2: track 31.2 -> 15.1 mm, vias 2 -> 1
- net Net-(J4-Pin_1): track 11.4 -> 27.4 mm, vias 0 -> 1
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- removed copper zone on B.Cu, net +3V3
- removed copper zone on F.Cu, net +3V3
- removed copper zone on B.Cu, net GND
Other:
- board size 51 x 51 mm -> 30.5 x 51 mm
- board text added: "Boot Switch"
- board text added: "Oi note to me. Try to add the loewr moutning holes of the camera so we can do spacers AND"
- board text added: "m3 mounting holes ON ALL"
- board text added: "reduce board size to 30.5mm if possible"

Commit message: Full final layout. A little over 2sq Inches
Parts:
- added ?: , , F.Cu at (140.5, 106.0)
- added ?: , , F.Cu at (132.4, 138.2)
- added ?: , , F.Cu at (140.5, 103.5)
- added D2: LED, Footprint:LEDIndicator, F.Cu at (113.4, 143.8)
- added R6: 160hm, Footprint:RESIndicatpr, F.Cu at (120.3, 138.0)
- added REF**: TestPoint_2Pads_Pitch2.54mm_Drill0.8mm, TestPoint:TestPoint_2Pads_Pitch2.54mm_Drill0.8mm, F.Cu at (113.1, 102.6)
- added U4: MCP73832T-2ACI/OT, Footprint:SOT-23-5_MC_MCH, F.Cu at (122.9, 146.3)
- C4, C5: moved to B.Cu
- D4, D5, R12, R13: moved to F.Cu
- J3: footprint Footprint:CONN2_B2B-PH-K-S_JST -> Footprint:CONN_S2B-XH-A_JST
- moved C4 41.9 mm to (125.7, 112.6), turned to 0 degrees
- moved C5 40.6 mm to (125.7, 114.7)
- moved C13 22.6 mm to (118.2, 144.0), turned to 0 degrees
- moved SW2 20.8 mm to (113.3, 138.9), turned to 90 degrees
- moved D6 13.4 mm to (129.6, 131.2), turned to 90 degrees
- moved C8 10.2 mm to (126.3, 149.7), turned to 90 degrees
- moved R12 9.61 mm to (125.2, 143.4), turned to 180 degrees
- moved C12 8.81 mm to (128.9, 142.2)
- moved D4 8.62 mm to (125.2, 141.8), turned to 0 degrees
- moved SW3 6.10 mm to (131.2, 149.5)
- moved R17 4.66 mm to (119.6, 141.1), turned to -90 degrees
- moved D1 4.36 mm to (131.9, 144.8)
- moved C9 3.87 mm to (112.5, 126.4)
- moved Q1 3.61 mm to (134.1, 140.6), turned to 90 degrees
- moved D5 3.46 mm to (121.1, 142.7), turned to 90 degrees
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Connections:
- U2 pad 30: unconnected-(U2-IO37-Pad30) -> Net-(U2-IO37)
Routing:
- net +3V3: track 6.19 -> 126.7 mm, vias 0 -> 8
- net GND: track 11.3 -> 59.5 mm, vias 0 -> 6
- net /SDA: track 31.4 -> 61.5 mm, vias 2 -> 3
- net /SCL: track 39.1 -> 64.0 mm
- net /D2: track 15.1 -> 25.9 mm, vias 1 -> 3
- net Net-(SW2A-B): track 20.8 -> 11.1 mm
- net Net-(D2-A): track 0.00 -> 9.27 mm
- net Net-(D1-A): track 12.0 -> 5.21 mm
- net Net-(JP2-B): track 5.39 -> 11.9 mm, vias 0 -> 1
- net Net-(D4-A): track 32.8 -> 38.5 mm, vias 0 -> 1
- net Net-(J4-Pin_1): track 27.4 -> 22.2 mm, vias 1 -> 2
- net Net-(SW3A-B): track 33.8 -> 38.0 mm
- net Net-(J3-Pin_2): track 5.76 -> 8.82 mm
- net Net-(U2-IO37): track 0.00 -> 2.89 mm
- net Net-(D1-K): track 13.6 -> 16.0 mm
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- added copper zone on B.Cu, net +3V3
- added copper zone on B.Cu, net GND
- added copper zone on F.Cu, net GND
Other:
- outline, holes or cut-outs redrawn
- board text added: "Hope Haptics 2025 Janus Sucharitakul Brandon Allen"
- board text added: "Test 3v3"
- board text added: "Test GND"
- board text added: "Test SCL"
- board text added: "Test SDA"
- board text added: "Test the schottky diode V drop"
- board text removed: "3V3 test"
- board text removed: "5V test"
- board text removed: "Boot Switch"
- board text removed: "Oi note to me. Try to add the loewr moutning holes of the camera so we can do spacers AND"
- board text removed: "m3 mounting holes ON ALL"
- board text removed: "reduce board size to 30.5mm if possible"
